Commit message: widespread updates to get navigator working with the carla_interface

File: data/carla.urdf (robot description, URDF)
Before this commit: robot carla-bopp, 3 links, 2 joints
Links:
- link model_link: geometry visual mesh filename=file:///carla_interface/data/hailbopp.stl scale=1.0 1.0 1.0

Commit message: added a rear facing camera and set it so that navigator would launch rviz

File: data/carla.urdf (robot description, URDF)
Before this commit: robot carla-bopp, 3 links, 2 joints
Links:
- link model_link: geometry visual mesh filename=file:///navigator/data/hailbopp.stl scale=1.0 1.0 1.0
